File: PCB/Joker60-NoArrows.kicad_pcb (KiCad board)
At the start: 2 copper layers, 283 x 94.2 mm, 244 parts, among them J1 TYPE-C-31-M12_13, J2 Conn_01x14, J3 Conn_ARM_JTAG_SWD_10, SW1 ESC, SW10 9, SW100 SPACE_625, SW101 HENKAN_100, SW102 RALT_100, SW103 RALT_100, SW104 RGUI_100, SW105 RCTRL_100, SW106 LGUI_100, SW107 LALT_125, SW108 MUHENKAN_100, SW109 SPACE_450, SW11 0, SW110 HENKAN_125, SW111 HENKAN_125, SW112 HENKAN_125, SW113 RALT_100, SW114 RALT_125, SW115 RCTRL_100, SW116 RCTRL_100, SW117 RCTRL_100, SW12 -_, SW13 +=, SW14 2U BKSP, SW15 TAB_150, SW16 Q, SW17 W, SW18 E, SW19 R, SW2 1, SW20 T, SW21 Y, SW22 U, SW23 I, SW24 O, SW25 P, SW26 [{, SW27 ]}, SW28 1U_RBKSP, SW29 CAPS_175, SW3 2, SW30 A, SW31 S, SW32 D, SW33 F, SW34 G, SW35 H, SW36 J, SW37 K, SW38 L, SW39 :;, SW4 3, SW40 @', SW41 ~~#, SW42 LSHIFT_125, SW43 |\, SW44 Z, SW45 X, SW46 C, SW47 V, SW48 B, SW49 N, SW5 4, SW50 M, SW51 <,, SW52 >., SW53 ?/, SW54 LCTRL_100, SW55 LGUI_125, SW56 LALT_100, SW57 SPACE_275, SW58 RALT_125, SW59 RGUI_125, SW6 5, SW60 RCTRL_125, SW61 LGUI_125, SW62 LALT_125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

Commit message: 2/12/221
Parts:
- removed G3: Acheron Logo, acheron_Logos:acheronLong
- removed G4: Doddle60Label, doddle60Graphics:doddle60Label
- removed G5: LabelMask, doddle60Graphics:doddle60LabelMask
- RCC1, RCC2, RL1, RPU1, RRST1, RSH1, RSH2, RSI1, RSO1, RVDD1: footprint acheron_Components:R_SMD_1026 -> acheron_Components:R_SMD_1206
Routing:
- net Row3: track 280.4 -> 317.0 mm
- net Net-(DRST1-Pad2): track 376.7 -> 386.2 mm
- net GND: track 406.0 -> 413.2 mm, vias 20 -> 24
- net Col7: track 599.8 -> 603.8 mm
- net Row5: track 418.0 -> 420.0 mm
- net Net-(D65-Pad2): track 52.6 -> 53.5 mm
- net Col6: track 475.3 -> 476.1 mm
Other:
- board text removed: "(I) If you want to check or reroute a specific trace, it is recommended that you use the High Contrast mode. Turn it on at View > Contrast mode > Check "High Contrast Mode". The icon is also available at the left icon column."
- board text removed: "(II) It is recommended that the user has some knowledge in Git usage, since it is the main VCS tool used for the Acheron Project."
- board text removed: "(III) All footprints are available either through KiCad's native libraries or the Acheron Library (http://github.com/Gondolindrim/AcheronLibrary). To facilitate the portability of the Acheron projects, this library is generally added at the ${KIPRJMOD} folder as a Git submodule. Hence, right after cloning the PCB repository, run: $ git submodule init --update To update the submodules."
- board text removed: "(IV) For detailed information, check the Acheron Docs page for the ArcticPCB: http://gondolindrim.github.io/AcheronDocs/arctic/intro.html"
- board text removed: "(i) The grid unit (1U) value used was 3/4" = 19.05mm"
- board text removed: "(ii) The PCB was designed to fit the standards of the PCBWay manufacturer, at their cheapest settings."
- board text removed: "(iii) All parts were quoted on the LCSC supplier (https://lcsc.com)."
- board text removed: "(iv) You can always contact Gondolindrim through:"
- board text removed: "(v) Most manufacturers list minimum character height as 0.8mm, and warn that any words using values below that will be undiscernable or unreadable. I have found that values down to 0.6mm (25 thou) can be used, although at that level a really close look is needed. Indeed, the minimum character height at which characters are easily readable is 0.8mm"
- board text removed: "- ArcticPCB's GitHub page: http://github.com/Gondolindrim/ArcticPCB"
- board text removed: "- Discord: Gondolindrim#9738"
- board text removed: "- E-mail: alvaro.augusto.volpato@gmail.com"
- board text removed: "- Reddit: /u/gondolindrim"
- board text removed: "Also be sure to check with your parts supplier if they have all the necessary parts in the Bill of Materials and change parts and footprints accordingly to availability"
- board text removed: "Be aware that capabilities may vary among manufacturers, so be sure to check with your manufacturer if they support the minimum values used."
- board text removed: "GENERAL OBSERVATIONS"
- board text removed: "MINIMUM CLEARANCE: 6 thou"
- board text removed: "MINIMUM CLEARANCE: 8 thou"
- board text removed: "MINIMUM VALUES"
- board text removed: "RECOMMENDED VALUES"
- board text removed: "SILKSCREEN CHARACTER HEIGHT: 25 thou (see General Observation (v))"
- board text removed: "SILKSCREEN CHARACTER HEIGHT: 32 thou"
- board text removed: "SILKSCREEN CHARACTER TRACE WIDTH: 6 thou"
- board text removed: "SILKSCREEN CHARACTER TRACE WIDTH: 8 thou"
- board text removed: "TRACE WIDTH: 10 thou"
- board text removed: "TRACE WIDTH: 6 thou (approx. 0.15 mm)"
- board text removed: "TRACE-TO-EDGE AND VIA-TO-EDGE DISTANCE: 8 thou"
- board text removed: "These are general hints to use this PCB file. They are aimed specially at thoise new to KiCad or ECAD in general and to whoever wishes to use this project."
- board text removed: "These values were the default values used when possible."
- board text removed: "USAGE GUIDE (PLEASE READ)"
- board text removed: "VIA DIAMETER: 20 thou (approx. 0.5mm)"
- board text removed: "VIA DIAMETER: 32 thou (approx. 0.8mm)"
- board text removed: "VIA HOLE SIZE: 12 thou (approx. 0.3mm)"
- board text removed: "VIA HOLE SIZE: 16 thou (approx. 0.4mm)"
- board text removed: "VIA-TO-VIA AND VIA-TO-TRACE CLEARANCE: 6 thou"
- board text removed: "VIA-TO-VIA AND VIA-TO-TRACE CLEARANCE: 8 thou"

Commit message: 8/29
Parts:
- removed CB1, CB4, CB6: 1µ, Capacitor_SMD:C_0402_1005Metric
- removed CB10, CB9: 1µ, Capacitor_SMD:C_0805_2012Metric
- removed CB2, CB3, CB5, CB8: 100n, Capacitor_SMD:C_0402_1005Metric
- removed CB7: 100nF, Capacitor_SMD:C_0402_1005Metric
- removed CRST1: 10u, Capacitor_SMD:C_0805_2012Metric_Pad1.15x1.40mm_HandSolder
- removed CRST2: 4.7n, Capacitor_SMD:C_0805_2012Metric_Pad1.15x1.40mm_HandSolder
- removed CSH1, CSH2: 4.7nF, Capacitor_SMD:C_0805_2012Metric
- removed CSI1, CSO1: 1µ, Capacitor_SMD:C_0805_2012Metric_Pad1.15x1.40mm_HandSolder
- removed CUSB1: 100n, Capacitor_SMD:C_0805_2012Metric_Pad1.15x1.40mm_HandSolder
- removed DF1: SMF9.0CA, acheron_Components:D_SOD-123_Bidirectional
- removed DL1: 19-217/R6C-AL1M2VY/3T, LED_SMD:LED_0603_1608Metric
- removed DRST1: B0520LW, acheron_Components:D_SOD-123
- removed DS1, DSH1: RB060M-60TR, acheron_Components:D_SOD-123
- removed H4: Oval Mounting Hole, acheron_MountingHoles:MoutingHole_Oval_7mm_5.0x2.5mm
- removed J1: TYPE-C-31-M12_13, acheron_Connectors:TYPE-C-31-M-12
- removed J3: Conn_ARM_JTAG_SWD_10, acheron_Connectors:Conn_ARM_JTAG_SWD_10
- removed L1: ACM2012-900-2P-T002, acheron_Components:ACM2012-2P
- removed L2: MGFL1608F1R0MT-LF, Inductor_SMD:L_0603_1608Metric
- removed L3: CMI322513U1R0KT, Inductor_SMD:L_1210_3225Metric
- removed QRST1: DTC123J, Package_TO_SOT_SMD:SOT-23
- removed RL1: 620R, acheron_Components:R_SMD_1206
- removed RPU1: 1.5k, acheron_Components:R_SMD_1206
- removed RRST1, RSI1, RSO1: 100k, acheron_Components:R_SMD_1206
- removed RSH1, RSH2: 1M, acheron_Components:R_SMD_1206
- removed RVDD1: R010 1%, acheron_Components:R_SMD_1206
- removed SW1: ESC, acheron_MX_SolderMask:MX100
- removed SWRST1: SW_Push, acheron_Hardware:smdPushBtn
- removed U3: MCP1700-3302E_SOT23, Package_TO_SOT_SMD:SOT-23
- added C1: 1uF, Capacitor_SMD:C_0603_1608Metric, F.Cu at (325.6, 114.6)
- added C2: 0.1uF, Capacitor_SMD:C_0603_1608Metric, F.Cu at (332.1, 127.2)
- added C3: 0.1uF, Capacitor_SMD:C_0603_1608Metric, F.Cu at (321.5, 126.9)
- added C4: 0.1uF, Capacitor_SMD:C_0603_1608Metric, F.Cu at (320.4, 118.7)
- added C5: 10uF, Capacitor_SMD:C_0603_1608Metric, F.Cu at (331.3, 116.4)
- added R1: 22Ω, Resistor_SMD:R_0603_1608Metric, F.Cu at (329.3, 116.3)
- added R2: 22Ω, Resistor_SMD:R_0603_1608Metric, F.Cu at (327.4, 116.3)
- added R3: 10kΩ, Resistor_SMD:R_0603_1608Metric, F.Cu at (321.4, 117.1)
- added R4: 10kΩ, Resistor_SMD:R_0603_1608Metric, F.Cu at (329.8, 129.5)
- added SW118: SW_PUSH, random-keyboard-parts:SKQG-1155865, F.Cu at (351.4, 106.7)
- added USB1: HRO-TYPE-C-31-M-12, Keebio-Parts:HRO-TYPE-C-31-M-12-Assembly, F.Cu at (337.7, 81.5)
- added Y1: Resonator_Small, proj_local:Resonator_SMD_muRata_CSTxExxV-3Pin_3.0x1.1mm_HandSoldering_Compact, F.Cu at (315.9, 118.2)
- F1: value 1A trip PTC -> Polyfuse_Small; footprint acheron_Components:Fuse_1812_4532 -> Fuse:Fuse_0805_2012Metric
- J2: value Conn_01x14 -> Conn_02x03_Odd_Even; footprint acheron_Connectors:PinHeader_1x14_P2.54mm_Vertical -> Connector_PinHeader_2.54mm:PinHeader_2x03_P2.54mm_Vertical
- RCC1, RCC2: footprint acheron_Components:R_SMD_1206 -> Resistor_SMD:R_0805_2012Metric
- SW96: footprint acheron_MX_SolderMask:MX200R -> acheron_MX_SolderMask:MX200
- U1: value STM32F072-LQFP48 -> SRV05-4; footprint acheron_Components:LQFP-48_7x7mm_P0.5mm -> Package_TO_SOT_SMD:SOT-23-6
- U2: value USBLC6-2SC6 -> ATmega32U4-MU; footprint acheron_Components:SOT-23-6 -> Package_DFN_QFN:QFN-44-1EP_7x7mm_P0.5mm_EP5.2x5.2mm
- moved U2 27.2 mm to (326.7, 122.7), turned to 270 degrees
- moved U1 22.9 mm to (336.3, 98.9), turned to 180 degrees
- moved RCC2 10.7 mm to (341.1, 94.7), turned to 180 degrees
- moved F1 5.97 mm to (336.4, 96.0), turned to 180 degrees
- moved J2 3.11 mm to (349.7, 115.5)
- moved RCC1 1.57 mm to (332.2, 94.9)
- turned SW103 to 180 degrees
- turned SW111 to 180 degrees
- turned SW115 to 180 degrees
- turned SW58 to 180 degrees
- turned SW59 to 180 degrees
- turned SW62 to 180 degrees
- turned SW74 to 180 degrees
- turned SW75 to 180 degrees
- turned SW80 to 180 degrees
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Connections:
- F1 pad 1: Net-(DF1-Pad1) -> +5V
- J2 pad 1: Extra1 -> Col13
- J2 pad 2: Extra2 -> +5V
- J2 pad 3: Extra3 -> Row1
- J2 pad 4: Extra4 -> Col14
- J2 pad 5: Extra5 -> Net-(J2-Pad5)
- J2 pad 6: Extra6 -> GND
- U1 pad 1: VDD -> D-
- U1 pad 2: Col12 -> GND
- U1 pad 3: Col11 -> Net-(U1-Pad3)
- U1 pad 4: Col10 -> Net-(U1-Pad4)
- U1 pad 5: Col9 -> VBUS
- U1 pad 6: Col8 -> D+
- U2 pad 2: GND -> +5V
- U2 pad 4: DBus- -> Net-(R2-Pad1)
- U2 pad 5: VBUS -> GND
- U2 pad 6: DBus+ -> Net-(C1-Pad1)
Routing:
- net Net-(DRST1-Pad2): track 386.2 -> 0.00 mm
- net NRST: track 173.9 -> 0.00 mm, vias 4 -> 0
- net 3.3V: track 173.2 -> 0.00 mm, vias 3 -> 0
- net GND: track 413.2 -> 279.1 mm
- net BOOT0: track 131.4 -> 0.00 mm, vias 2 -> 0
- net +5V: track 0.00 -> 129.1 mm, vias 0 -> 5
- net 5V: track 95.4 -> 0.00 mm, vias 2 -> 0
- net SWDIO: track 90.9 -> 0.00 mm, vias 1 -> 0
- net SWCLK: track 90.8 -> 0.00 mm, vias 1 -> 0
- net VDD: track 69.0 -> 0.00 mm, vias 6 -> 0
- net Net-(J2-Pad5): track 0.00 -> 66.8 mm, vias 0 -> 2
- net Extra14: track 41.2 -> 0.00 mm
- net Col13: track 341.1 -> 381.2 mm, vias 0 -> 1
- net Col14: track 399.1 -> 436.3 mm, vias 0 -> 1
- net Extra13: track 36.0 -> 0.00 mm
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- added copper zone on B.Cu, net (none)
- added copper zone on F.Cu, net (none)
- removed copper zone on B.Cu, net /SHIELD
- removed copper zone on F.Cu, net GNDD
- removed copper zone on B.Cu, net VDD
Other:
- rule trace_min: 0.254 -> 0.25
- board text added: "6.490009843 x 6.587918307 Hole H4"

Commit message: 10/7
Parts:
- added SW1: ESC, acheron_MX_SolderMask:MX100, F.Cu at (346.2, 91.4)
Connections:
- D1 pad 1: Row1 -> Row0
- D10 pad 1: Row1 -> Row0
- D11 pad 1: Row1 -> Row0
- D12 pad 1: Row1 -> Row0
- D13 pad 1: Row1 -> Row0
- D14 pad 1: Row1 -> Row0
- D15 pad 1: Row2 -> Row1
- D16 pad 1: Row2 -> Row1
- D17 pad 1: Row2 -> Row1
- D18 pad 1: Row2 -> Row1
- D19 pad 1: Row2 -> Row1
- D2 pad 1: Row1 -> Row0
- D20 pad 1: Row2 -> Row1
- D21 pad 1: Row2 -> Row1
- D22 pad 1: Row2 -> Row1
- D23 pad 1: Row2 -> Row1
- D24 pad 1: Row2 -> Row1
- D25 pad 1: Row2 -> Row1
- D26 pad 1: Row2 -> Row1
- D27 pad 1: Row2 -> Row1
- D28 pad 1: Row2 -> Row1
- D29 pad 1: Row3 -> Row2
- D3 pad 1: Row1 -> Row0
- D30 pad 1: Row3 -> Row2
- D31 pad 1: Row3 -> Row2
- D32 pad 1: Row3 -> Row2
- D33 pad 1: Row3 -> Row2
- D34 pad 1: Row3 -> Row2
- D35 pad 1: Row3 -> Row2
- D36 pad 1: Row3 -> Row2
- D37 pad 1: Row3 -> Row2
- D38 pad 1: Row3 -> Row2
- D39 pad 1: Row3 -> Row2
- D4 pad 1: Row1 -> Row0
- D40 pad 1: Row3 -> Row2
- D41 pad 1: Row3 -> Row2
- D42 pad 1: Row4 -> Row3
- D43 pad 1: Row4 -> Row3
- D44 pad 1: Row4 -> Row3
- D45 pad 1: Row4 -> Row3
- D46 pad 1: Row4 -> Row3
- D47 pad 1: Row4 -> Row3
- D48 pad 1: Row4 -> Row3
- D49 pad 1: Row4 -> Row3
- D5 pad 1: Row1 -> Row0
- D50 pad 1: Row4 -> Row3
- D51 pad 1: Row4 -> Row3
- D52 pad 1: Row4 -> Row3
- D53 pad 1: Row4 -> Row3
- D54 pad 1: Row5 -> Row4
- D55 pad 1: Row5 -> Row4
- D56 pad 1: Row5 -> Row4
- D57 pad 1: Row5 -> Row4
- D58 pad 1: Row5 -> Row4
- D59 pad 1: Row5 -> Row4
- D6 pad 1: Row1 -> Row0
- D60 pad 1: Row5 -> Row4
- D61 pad 1: Row5 -> Row4
- D62 pad 1: Row4 -> Row3
- D63 pad 1: Row4 -> Row3
- D64 pad 1: Row5 -> Row4
- D65 pad 1: Row3 -> Row2
- D66 pad 1: Row5 -> Row4
- D67 pad 1: Row5 -> Row4
- D68 pad 1: Row2 -> Row1
- D69 pad 1: Row5 -> Row4
- D7 pad 1: Row1 -> Row0
- D70 pad 1: Row5 -> Row4
- D8 pad 1: Row1 -> Row0
- D9 pad 1: Row1 -> Row0
- J2 pad 1: Col13 -> Col12
- J2 pad 3: Row1 -> Row0
- J2 pad 4: Col14 -> Col13
- SW10 pad 1: Col10 -> Col9
- SW100 pad 1: Col7 -> Col6
- SW101 pad 1: Col10 -> Col9
- SW102 pad 1: Col11 -> Col10
- SW103 pad 1: Col12 -> Col11
- SW104 pad 1: Col13 -> Col12
- SW105 pad 1: Col14 -> Col13
- SW106 pad 1: Col2 -> Col1
- SW107 pad 1: Col3 -> Col2
- SW108 pad 1: Col4 -> Col3
- SW109 pad 1: Col7 -> Col6
- SW11 pad 1: Col11 -> Col10
- SW110 pad 1: Col9 -> Col8
- SW111 pad 1: Col10 -> Col9
- SW112 pad 1: Col11 -> Col10
- SW113 pad 1: Col12 -> Col11
- SW114 pad 1: Col14 -> Col13
- SW115 pad 1: Col12 -> Col11
- SW116 pad 1: Col13 -> Col12
- SW117 pad 1: Col14 -> Col13
- SW12 pad 1: Col12 -> Col11
- SW13 pad 1: Col13 -> Col12
- SW14 pad 1: Col14 -> Col13
- SW15 pad 1: Col1 -> Col0
- SW16 pad 1: Col2 -> Col1
- SW17 pad 1: Col3 -> Col2
- SW18 pad 1: Col4 -> Col3
- SW19 pad 1: Col5 -> Col4
- SW2 pad 1: Col2 -> Col1
- SW20 pad 1: Col6 -> Col5
- SW21 pad 1: Col7 -> Col6
- SW22 pad 1: Col8 -> Col7
- SW23 pad 1: Col9 -> Col8
- SW24 pad 1: Col10 -> Col9
- SW25 pad 1: Col11 -> Col10
- SW26 pad 1: Col12 -> Col11
- SW27 pad 1: Col13 -> Col12
- SW28 pad 1: Col14 -> Col13
- SW29 pad 1: Col1 -> Col0
- SW3 pad 1: Col3 -> Col2
- SW30 pad 1: Col2 -> Col1
- SW31 pad 1: Col3 -> Col2
- SW32 pad 1: Col4 -> Col3
- SW33 pad 1: Col5 -> Col4
- SW34 pad 1: Col6 -> Col5
- SW35 pad 1: Col7 -> Col6
- SW36 pad 1: Col8 -> Col7
- SW37 pad 1: Col9 -> Col8
- SW38 pad 1: Col10 -> Col9
- SW39 pad 1: Col11 -> Col10
- SW4 pad 1: Col4 -> Col3
- SW40 pad 1: Col12 -> Col11
- SW41 pad 1: Col13 -> Col12
- SW42 pad 1: Col1 -> Col0
- SW43 pad 1: Col2 -> Col1
- SW44 pad 1: Col3 -> Col2
- SW45 pad 1: Col4 -> Col3
- SW46 pad 1: Col5 -> Col4
- SW47 pad 1: Col6 -> Col5
- SW48 pad 1: Col7 -> Col6
- SW49 pad 1: Col8 -> Col7
- SW5 pad 1: Col5 -> Col4
- SW50 pad 1: Col9 -> Col8
- SW51 pad 1: Col10 -> Col9
- SW52 pad 1: Col11 -> Col10
- SW53 pad 1: Col12 -> Col11
- SW54 pad 1: Col2 -> Col1
- SW55 pad 1: Col2 -> Col1
- SW56 pad 1: Col3 -> Col2
- SW57 pad 1: Col7 -> Col6
- SW58 pad 1: Col11 -> Col10
- SW59 pad 1: Col12 -> Col11
- SW6 pad 1: Col6 -> Col5
- SW60 pad 1: Col14 -> Col13
- SW61 pad 1: Col1 -> Col0
- SW62 pad 1: Col3 -> Col2
- SW63 pad 1: Col1 -> Col0
- SW64 pad 1: Col14 -> Col13
- SW65 pad 1: Col14 -> Col13
- SW66 pad 1: Col1 -> Col0
- SW67 pad 1: Col4 -> Col3
- SW68 pad 1: Col10 -> Col9
- SW69 pad 1: Col2 -> Col1
- SW7 pad 1: Col7 -> Col6
- SW70 pad 1: Col6 -> Col5
- SW71 pad 1: Col3 -> Col2
- SW72 pad 1: Col14 -> Col13
- SW73 pad 1: Col1 -> Col0
- SW74 pad 1: Col13 -> Col12
- SW75 pad 1: Col14 -> Col13
- SW76 pad 1: Col15 -> Col14
- SW77 pad 1: Col14 -> Col13
- SW78 pad 1: Col13 -> Col12
- SW79 pad 1: Col14 -> Col13
- SW8 pad 1: Col8 -> Col7
- SW80 pad 1: Col9 -> Col8
- SW81 pad 1: Col4 -> Col3
- SW82 pad 1: Col9 -> Col8
- SW83 pad 1: Col10 -> Col9
- SW84 pad 1: Col11 -> Col10
- SW85 pad 1: Col4 -> Col3
- SW86 pad 1: Col7 -> Col6
- SW87 pad 1: Col5 -> Col4
- SW88 pad 1: Col6 -> Col5
- SW89 pad 1: Col8 -> Col7
- SW9 pad 1: Col9 -> Col8
- SW90 pad 1: Col7 -> Col6
- SW91 pad 1: Col8 -> Col7
- SW92 pad 1: Col9 -> Col8
- SW93 pad 1: Col10 -> Col9
- SW94 pad 1: Col11 -> Col10
- SW95 pad 1: Col12 -> Col11
- SW96 pad 1: Col13 -> Col12
- SW97 pad 1: Col14 -> Col13
- SW98 pad 1: Col1 -> Col0
- SW99 pad 1: Col13 -> Col12
- U2 pad 10: Col14 -> Col13
- U2 pad 11: Col13 -> Col12
- U2 pad 12: Col12 -> Col11
- U2 pad 18: Col11 -> Col10
- U2 pad 19: Col10 -> Col9
- U2 pad 20: Col9 -> Col8
- U2 pad 21: Col8 -> Col7
- U2 pad 22: Col7 -> Col6
- U2 pad 25: Col6 -> Col5
- U2 pad 26: Col5 -> Col4
- U2 pad 27: Col4 -> Col3
- U2 pad 28: Col3 -> Col2
- U2 pad 29: Row3 -> Row2
- U2 pad 30: Row4 -> Row3
- U2 pad 31: Col1 -> Col0
- U2 pad 32: Row5 -> Row4
- U2 pad 39: Col2 -> Col1
- U2 pad 41: Row2 -> Row1
- U2 pad 8: Col15 -> Col14
- U2 pad 9: Row1 -> Row0
Routing:
- net Row0: track 0.00 -> 600.1 mm, vias 0 -> 3
- net Row5: track 408.8 -> 0.00 mm
- net Row1: track 600.1 -> 284.6 mm, vias 3 -> 2
- net Col15: track 272.4 -> 0.00 mm, vias 3 -> 0
- net Col5: track 273.9 -> 483.7 mm
- net Col0: track 0.00 -> 175.5 mm, vias 0 -> 1
- net Col14: track 436.3 -> 272.4 mm, vias 1 -> 3
- net Row4: track 281.8 -> 408.8 mm
- net Col6: track 483.7 -> 604.3 mm
- net Col2: track 152.5 -> 241.7 mm
- net Col3: track 241.7 -> 328.0 mm, vias 1 -> 0
- net Col10: track 490.0 -> 419.8 mm
- net Col13: track 381.2 -> 436.3 mm
- net Col4: track 328.0 -> 273.9 mm
- net Col9: track 530.6 -> 490.0 mm
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