File: PCB/Joker60-NoArrows.kicad_pcb (KiCad board)
At the start: 2 copper layers, 283 x 94.2 mm, 214 parts, among them J2 Conn_02x03_Odd_Even, SW1 ESC, SW10 9, SW100 SPACE_625, SW101 HENKAN_100, SW102 RALT_100, SW103 RALT_100, SW104 RGUI_100, SW105 RCTRL_100, SW106 LGUI_100, SW107 LALT_125, SW108 MUHENKAN_100, SW109 SPACE_450, SW11 0, SW110 HENKAN_125, SW111 HENKAN_125, SW112 HENKAN_125, SW113 RALT_100, SW114 RALT_125, SW115 RCTRL_100, SW116 RCTRL_100, SW117 RCTRL_100, SW118 SW_PUSH, SW12 -_, SW13 +=, SW14 2U BKSP, SW15 TAB_150, SW16 Q, SW17 W, SW18 E, SW19 R, SW2 1, SW20 T, SW21 Y, SW22 U, SW23 I, SW24 O, SW25 P, SW26 [{, SW27 ]}, SW28 1U_RBKSP, SW29 CAPS_175, SW3 2, SW30 A, SW31 S, SW32 D, SW33 F, SW34 G, SW35 H, SW36 J, SW37 K, SW38 L, SW39 :;, SW4 3, SW40 @', SW41 ~~#, SW42 LSHIFT_125, SW43 |\, SW44 Z, SW45 X, SW46 C, SW47 V, SW48 B, SW49 N, SW5 4, SW50 M, SW51 <,, SW52 >., SW53 ?/, SW54 LCTRL_100, SW55 LGUI_125, SW56 LALT_100, SW57 SPACE_275, SW58 RALT_125, SW59 RGUI_125, SW6 5, SW60 RCTRL_125, SW61 LGUI_125, SW62 LALT_125, SW63 STEPPED_CAPS_125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

Commit message: 12/20
Parts:
- moved D1 3.24 mm to (351.7, 98.3)
- moved RCC2 2.33 mm to (341.2, 97.1)
- turned SW1 to 180 degrees
Routing:
- net Col0: track 175.5 -> 153.4 mm
- net GND: track 279.1 -> 299.5 mm
- net Net-(D1-Pad2): track 5.38 -> 12.9 mm, vias 0 -> 1
- net Row0: track 600.1 -> 594.8 mm
- net Net-(RCC2-Pad2): track 6.04 -> 8.42 mm
