File: PCB/Joker60-NoArrows.sch (KiCad schematic (older format))
At the start: 246 parts, among them J1 TYPE-C-31-M12_13, J2 Conn_01x14, J3 Conn_ARM_JTAG_SWD_10, SW1 ESC, SW10 9, SW100 SPACE_625, SW101 HENKAN_100, SW102 RALT_100, SW103 RALT_100, SW104 RGUI_100, SW105 RCTRL_100, SW106 LGUI_100, SW107 LALT_125, SW108 MUHENKAN_100, SW109 SPACE_450, SW11 0, SW110 HENKAN_125, SW111 HENKAN_125, SW112 HENKAN_125, SW113 RALT_100, SW114 RALT_125, SW115 RCTRL_100, SW116 RCTRL_100, SW117 RCTRL_100, SW12 -_, SW13 +=, SW14 2U BKSP, SW15 TAB_150, SW16 Q, SW17 W, SW18 E, SW19 R, SW2 1, SW20 T, SW21 Y, SW22 U, SW23 I, SW24 O, SW25 P, SW26 [{, SW27 ]}, SW28 1U_RBKSP, SW29 CAPS_175, SW3 2, SW30 A, SW31 S, SW32 D, SW33 F, SW34 G, SW35 H, SW36 J, SW37 K, SW38 L, SW39 :;, SW4 3, SW40 @', SW41 ~~#, SW42 LSHIFT_125, SW43 |\\, SW44 Z, SW45 X, SW46 C, SW47 V, SW48 B, SW49 N, SW5 4, SW50 M, SW51 <,, SW52 >., SW53 ?/, SW54 LCTRL_100, SW55 LGUI_125, SW56 LALT_100, SW57 SPACE_275, SW58 RALT_125, SW59 RGUI_125, SW6 5, SW60 RCTRL_125, SW61 LGUI_125, SW62 LALT_125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

Commit message: 2/8/2021
Parts:
- CB1, CB4, CB6: LCSC Part# (none) -> C408910; Mfr (none) -> Walsin Tech Corp; Part# (none) -> 0402F105M6R3CT
- CB10, CB9: LCSC Part# (none) -> C92829; Mfr (none) -> Taiyo Yuden; Part# (none) -> TMK212BJ105KG-T
- CB2, CB3, CB5, CB8: LCSC Part# (none) -> C169292; Mfr (none) -> Vishay Intertech; Part# (none) -> VJ0402G104KXQCW1BC
- CB7: LCSC Part# (none) -> C301997; Mfr (none) -> Walsin Tech Corp; Part# (none) -> 0402X104K160CT
- CRST1: LCSC Part# (none) -> C40894; Mfr (none) -> FH(Guangdong Fenghua Advanced Tech); Part# (none) -> 0805X106K250NT
- CRST2, CSH1, CSH2: LCSC Part# (none) -> C50131; Mfr (none) -> Samsung Electro-Mechanics; Part# (none) -> CL21B472KBANNNC
- CSI1, CSO1: LCSC Part# (none) -> C77080; Mfr (none) -> Murata Electronics; Part# (none) -> GRM21BR71E105KA99L
- CUSB1: LCSC Part# (none) -> C49678; Mfr (none) -> YAGEO; Part# (none) -> CC0805KRX7R9BB104
- D1, D10, D11, D12, D13, D14, D15, D16, D17, D18, D19, D2, D20, D21, D22, D23, D24, D25, D26, D27, D28, D29, D3, D30, D31, D32, D33, D34, D35, D36, D37, D38, D39, D4, D40, D41, D42, D43, D44, D45, D46, D47, D48, D49, D5, D50, D51, D52, D53, D54, D55, D56, D57, D58, D59, D6, D60, D61, D62, D63, D64, D65, D66, D67, D68, D69, D7, D70, D8, D9: LCSC Part# (none) -> C444720; Mfr (none) -> Slkor(SLKORMICRO Elec.); Part# (none) -> 1N4148W
- DF1: LCSC Part# (none) -> C435473; Mfr (none) -> AnBon; Part# (none) -> SMF9.0CA
- DL1: LCSC Part# (none) -> C72044; Mfr (none) -> Everlight Elec; Part# (none) -> 19-217/R6C-AL1M2VY/3T
- DRST1: LCSC Part# (none) -> C8570; Mfr (none) -> Changjiang Electronics Tech (CJ); Part# (none) -> B0520LW
- DS1, DSH1: LCSC Part# (none) -> C114257; Mfr (none) -> ROHM Semicon; Part# (none) -> RB060M-60TR
- F1: LCSC Part# (none) -> C883140; Mfr (none) -> BHFUSE; Part# (none) -> BSMD1812-050-24V
- SWRST1: LCSC Part# (none) -> C221929; Mfr (none) -> C&K; Part# (none) -> RS-187R05A2-DSMTRT
- U1: LCSC Part# (none) -> C81720; Mfr (none) -> STMicroelectronics; Part# (none) -> STM32F072CBT6
- U2: LCSC Part# (none) -> C7519; Mfr (none) -> STMicroelectronics; Part# (none) -> USBLC6-2SC6
- U3: LCSC Part# (none) -> C39051; Mfr (none) -> Microchip Tech; Part# (none) -> MCP1700T-3302E/TT

Commit message: 2/12/221
Parts:
- J1: LCSC Part# (none) -> C223906; Mfr (none) -> Korean Hroparts Elec; Part# (none) -> TYPE-C-31-M-13
- L1: LCSC Part# (none) -> C19972; Mfr (none) -> TDK; Part# (none) -> ACM2012-900-2P-T002
- L2: LCSC Part# (none) -> C281108; Mfr (none) -> microgate; Part# (none) -> MGFL1608F1R0MT-LF
- L3: LCSC Part# (none) -> C99412; Mfr (none) -> FH(Guangdong Fenghua Advanced Tech); Part# (none) -> CMI322513U1R0KT
- QRST1: LCSC Part# (none) -> C111724; Mfr (none) -> ROHM Semicon; Part# (none) -> DTC123JKAT146
- RCC1, RCC2: footprint acheron_Components:R_SMD_1026 -> acheron_Components:R_SMD_1206; LCSC Part# (none) -> C351456; Mfr (none) -> Resistor.Today; Part# (none) -> PTFR1206B5K10P9
- RL1: footprint acheron_Components:R_SMD_1026 -> acheron_Components:R_SMD_1206; LCSC Part# (none) -> C25391; Mfr (none) -> UNI-ROYAL(Uniroyal Elec); Part# (none) -> 1206W4J0621T5E
- RPU1: footprint acheron_Components:R_SMD_1026 -> acheron_Components:R_SMD_1206; LCSC Part# (none) -> C114929; Mfr (none) -> YAGEO; Part# (none) -> RC1206FR-071K5L
- RRST1, RSI1, RSO1: footprint acheron_Components:R_SMD_1026 -> acheron_Components:R_SMD_1206; LCSC Part# (none) -> C346155; Mfr (none) -> KOA Speer Elec; Part# (none) -> RN73H2BTTD1003B25
- RSH1, RSH2: footprint acheron_Components:R_SMD_1026 -> acheron_Components:R_SMD_1206; LCSC Part# (none) -> C325894; Mfr (none) -> TyoHM; Part# (none) -> RMC12061M1%N
- RVDD1: footprint acheron_Components:R_SMD_1026 -> acheron_Components:R_SMD_1206; LCSC Part# (none) -> C104920; Mfr (none) -> RALEC; Part# (none) -> RTT06R010FTP
Changed lines of the file:
@@
 F 0 "RRST1" V 10150 17725 31  0000 L CNN
 F 1 "100k" V 10225 17750 31  0000 L CNN
-F 2 "acheron_Components:R_SMD_1026" H 10225 17800 50  0001 C CNN
-F 3 "~" H 10225 17800 50  0001 C CNN
+F 2 "acheron_Components:R_SMD_1206" H 10225 17800 50  0001 C CNN
+F 3 "https://datasheet.lcsc.com/szlcsc/1912111437_KOA-Speer-Elec-RN73H2BTTD1003B25_C346155.pdf" H 10225 17800 50  0001 C CNN
+F 4 "C346155" H 10225 17800 50  0001 C CNN "LCSC Part#"
+F 5 "	KOA Speer Elec" H 10225 17800 50  0001 C CNN "Mfr"
+F 6 "RN73H2BTTD1003B25" H 10225 17800 50  0001 C CNN "Part#"
 	1    10225 17800
 	1    0    0    -1
@@
 F 1 "DTC123J" V 9959 17100 50  0000 C CNN
 F 2 "Package_TO_SOT_SMD:SOT-23" H 9725 17100 50  0001 L CNN
-F 3 "" H 9725 17100 50  0001 L CNN
+F 3 "https://datasheet.lcsc.com/szlcsc/1808272202_ROHM-Semicon-DTC123JKAT146_C111724.pdf" H 9725 17100 50  0001 L CNN
+F 4 "C111724" H 9725 17100 50  0001 C CNN "LCSC Part#"
+F 5 "ROHM Semicon" H 9725 17100 50  0001 C CNN "Mfr"
+F 6 "DTC123JKAT146" H 9725 17100 50  0001 C CNN "Part#"
 	1    9725 17100
 	0    1    -1   0
@@
 F 1 "TYPE-C-31-M12_13" H 6400 19000 50  0000 C CNN
 F 2 "acheron_Connectors:TYPE-C-31-M-12" V 5900 17725 50  0001 C CNN
-F 3 "https://www.usb.org/sites/default/files/documents/usb_type-c.zip" H 6600 17725 50  0001 C CNN
+F 3 "https://datasheet.lcsc.com/szlcsc/1811101526_Korean-Hroparts-Elec-TYPE-C-31-M-13_C223906.pdf" H 6600 17725 50  0001 C CNN
+F 4 "C223906" H 6400 17675 50  0001 C CNN "LCSC Part#"
+F 5 "Korean Hroparts Elec" H 6400 17675 50  0001 C CNN "Mfr"
+F 6 "	TYPE-C-31-M-13" H 6400 17675 50  0001 C CNN "Part#"
 	1    6400 17675
 	1    0    0    -1
@@
 F 0 "RSH1" H 6159 19356 31  0000 L CNN
 F 1 "1M" H 6159 19294 31  0000 L CNN
-F 2 "acheron_Components:R_SMD_1026" H 6100 19325 50  0001 C CNN
-F 3 "~" H 6100 19325 50  0001 C CNN
+F 2 "acheron_Components:R_SMD_1206" H 6100 19325 50  0001 C CNN
+F 3 "https://datasheet.lcsc.com/szlcsc/1912111437_TyoHM-RMC12061M1-N_C325894.pdf" H 6100 19325 50  0001 C CNN
+F 4 "C325894" H 6100 19325 50  0001 C CNN "LCSC Part#"
+F 5 "TyoHM" H 6100 19325 50  0001 C CNN "Mfr"
+F 6 "RMC12061M1%N" H 6100 19325 50  0001 C CNN "Part#"
 	1    6100 19325
 	1    0    0    -1
@@
 F 0 "RCC1" V 7075 17225 31  0000 C CNN
 F 1 "5.1k" V 7150 17225 31  0000 C CNN
-F 2 "acheron_Components:R_SMD_1026" H 7150 17225 50  0001 C CNN
-F 3 "~" H 7150 17225 50  0001 C CNN
+F 2 "acheron_Components:R_SMD_1206" H 7150 17225 50  0001 C CNN
+F 3 "https://datasheet.lcsc.com/szlcsc/2004211006_Resistor-Today-PTFR1206B5K10P9_C351456.pdf" H 7150 17225 50  0001 C CNN
+F 4 "C351456" H 7150 17225 50  0001 C CNN "LCSC Part#"
+F 5 "Resistor.Today" H 7150 17225 50  0001 C CNN "Mfr"
+F 6 "	PTFR1206B5K10P9" H 7150 17225 50  0001 C CNN "Part#"
 	1    7150 17225
 	0    1    1    0
@@
 F 0 "RSH2" H 1934 16881 31  0000 L CNN
 F 1 "1M" H 1934 16819 31  0000 L CNN
-F 2 "acheron_Components:R_SMD_1026" H 1875 16850 50  0001 C CNN
-F 3 "~" H 1875 16850 50  0001 C CNN
+F 2 "acheron_Components:R_SMD_1206" H 1875 16850 50  0001 C CNN
+F 3 "https://datasheet.lcsc.com/szlcsc/1912111437_TyoHM-RMC12061M1-N_C325894.pdf" H 1875 16850 50  0001 C CNN
+F 4 "C325894" H 1875 16850 50  0001 C CNN "LCSC Part#"
+F 5 "TyoHM" H 1875 16850 50  0001 C CNN "Mfr"
+F 6 "RMC12061M1%N" H 1875 16850 50  0001 C CNN "Part#"
 	1    1875 16850
 	1    0    0    -1
@@
 F 0 "RCC2" V 7075 17025 31  0000 C CNN
 F 1 "5.1k" V 7150 17025 31  0000 C CNN
-F 2 "acheron_Components:R_SMD_1026" H 7150 17025 50  0001 C CNN
-F 3 "~" H 7150 17025 50  0001 C CNN
+F 2 "acheron_Components:R_SMD_1206" H 7150 17025 50  0001 C CNN
+F 3 "https://datasheet.lcsc.com/szlcsc/2004211006_Resistor-Today-PTFR1206B5K10P9_C351456.pdf" H 7150 17025 50  0001 C CNN
+F 4 "C351456" H 7150 17025 50  0001 C CNN "LCSC Part#"
+F 5 "Resistor.Today" H 7150 17025 50  0001 C CNN "Mfr"
+F 6 "	PTFR1206B5K10P9" H 7150 17025 50  0001 C CNN "Part#"
 	1    7150 17025
 	0    1    1    0
@@
 F 0 "RSI1" V 10000 19925 31  0000 C CNN
 F 1 "100k" V 10075 19925 31  0000 C CNN
-F 2 "acheron_Components:R_SMD_1026" H 10075 19925 50  0001 C CNN
-F 3 "~" H 10075 19925 50  0001 C CNN
+F 2 "acheron_Components:R_SMD_1206" H 10075 19925 50  0001 C CNN
+F 3 "https://datasheet.lcsc.com/szlcsc/1912111437_KOA-Speer-Elec-RN73H2BTTD1003B25_C346155.pdf" H 10075 19925 50  0001 C CNN
+F 4 "	C346155" H 10075 19925 50  0001 C CNN "LCSC Part#"
+F 5 "KOA Speer Elec" H 10075 19925 50  0001 C CNN "Mfr"
+F 6 "RN73H2BTTD1003B25" H 10075 19925 50  0001 C CNN "Part#"
 	1    10075 19925
 	1    0    0    -1
@@
 F 0 "RSO1" V 11100 19925 31  0000 C CNN
 F 1 "100k" V 11175 19925 31  0000 C CNN
-F 2 "acheron_Components:R_SMD_1026" H 11175 19925 50  0001 C CNN
-F 3 "~" H 11175 19925 50  0001 C CNN
+F 2 "acheron_Components:R_SMD_1206" H 11175 19925 50  0001 C CNN
+F 3 "https://datasheet.lcsc.com/szlcsc/1912111437_KOA-Speer-Elec-RN73H2BTTD1003B25_C346155.pdf" H 11175 19925 50  0001 C CNN
+F 4 "	C346155" H 11175 19925 50  0001 C CNN "LCSC Part#"
+F 5 "KOA Speer Elec" H 11175 19925 50  0001 C CNN "Mfr"
+F 6 "RN73H2BTTD1003B25" H 11175 19925 50  0001 C CNN "Part#"
 	1    11175 19925
 	1    0    0    -1
@@
 F 0 "RPU1" V 7075 17975 31  0000 C CNN
 F 1 "1.5k" V 7150 17975 31  0000 C CNN
-F 2 "acheron_Components:R_SMD_1026" H 7150 17975 50  0001 C CNN
-F 3 "~" H 7150 17975 50  0001 C CNN
+F 2 "acheron_Components:R_SMD_1206" H 7150 17975 50  0001 C CNN
+F 3 "https://datasheet.lcsc.com/szlcsc/1810241211_YAGEO-RC1206FR-071K5L_C114929.pdf" H 7150 17975 50  0001 C CNN
+F 4 "C114929" H 7150 17975 50  0001 C CNN "LCSC Part#"
+F 5 "YAGEO" H 7150 17975 50  0001 C CNN "Mfr"
+F 6 "RC1206FR-071K5L" H 7150 17975 50  0001 C CNN "Part#"
 	1    7150 17975
 	0    1    1    0
@@
 F 1 "MGFL1608F1R0MT-LF" V 9868 19700 30  0000 C CNN
 F 2 "Inductor_SMD:L_0603_1608Metric" H 9750 19700 50  0001 C CNN
-F 3 "~" H 9750 19700 50  0001 C CNN
+F 3 "https://datasheet.lcsc.com/szlcsc/1811141852_microgate-MGFL1608F1R0MT-LF_C281108.pdf" H 9750 19700 50  0001 C CNN
+F 4 "C281108" H 9750 19700 50  0001 C CNN "LCSC Part#"
+F 5 "microgate" H 9750 19700 50  0001 C CNN "Mfr"
+F 6 "MGFL1608F1R0MT-LF" H 9750 19700 50  0001 C CNN "Part#"
 	1    9750 19700
 	0    -1   -1   0
@@
 F 1 "ACM2012-900-2P-T002" H 7225 15442 25  0000 C CNN
 F 2 "acheron_Components:ACM2012-2P" H 7225 15250 50  0001 C CNN
-F 3 "~" H 7225 15250 50  0001 C CNN
+F 3 "https://datasheet.lcsc.com/szlcsc/2006291108_TDK-ACM2012-900-2P-T002_C19972.pdf" H 7225 15250 50  0001 C CNN
+F 4 "C19972" H 7225 15250 50  0001 C CNN "LCSC Part#"
+F 5 "	TDK" H 7225 15250 50  0001 C CNN "Mfr"
+F 6 "ACM2012-900-2P-T002" H 7225 15250 50  0001 C CNN "Part#"
 	1    7225 15250
 	1    0    0    -1
 $EndComp
 $Comp
-L Joker60-NoArrows-rescue:R_Small-Device-doddle60-rescue RL1
-U 1 1 5E5122FD
-P 11950 19925
-F 0 "RL1" V 11875 19925 31  0000 C CNN
-F 1 "620R" V 11950 19925 31  0000 C CNN
-F 2 "acheron_Components:R_SMD_1026" H 11950 19925 50  0001 C CNN
-F 3 "~" H 11950 19925 50  0001 C CNN
-	1    11950 19925
-	1    0    0    -1
-$EndComp
-$Comp
 L Joker60-NoArrows-rescue:LED_Small-Device-doddle60-rescue DL1
 U 1 1 5E513BD6
@@
 F 1 "CMI322513U1R0KT" V 14093 14375 30  0000 C CNN
 F 2 "Inductor_SMD:L_1210_3225Metric" H 13975 14375 50  0001 C CNN
-F 3 "~" H 13975 14375 50  0001 C CNN
+F 3 "https://datasheet.lcsc.com/szlcsc/1811141420_FH-Guangdong-Fenghua-Advanced-Tech-CMI322513U1R0KT_C99412.pdf" H 13975 14375 50  0001 C CNN
+F 4 "C99412" H 13975 14375 50  0001 C CNN "LCSC Part#"
+F 5 "FH(Guangdong Fenghua Advanced Tech)" H 13975 14375 50  0001 C CNN "Mfr"
+F 6 "	CMI322513U1R0KT" H 13975 14375 50  0001 C CNN "Part#"
 	1    13975 14375
 	0    -1   -1   0
@@
 F 0 "RVDD1" V 13425 14575 31  0000 L CNN
 F 1 "R010 1%" V 13500 14650 15  0000 C CNN
-F 2 "acheron_Components:R_SMD_1026" H 13500 14650 50  0001 C CNN
-F 3 "~" H 13500 14650 50  0001 C CNN
+F 2 "acheron_Components:R_SMD_1206" H 13500 14650 50  0001 C CNN
+F 3 "https://datasheet.lcsc.com/szlcsc/1811081724_RALEC-RTT06R010FTP_C104920.pdf" H 13500 14650 50  0001 C CNN
+F 4 "C104920" H 13500 14650 50  0001 C CNN "LCSC Part#"
+F 5 "RALEC" H 13500 14650 50  0001 C CNN "Mfr"
+F 6 "RTT06R010FTP" H 13500 14650 50  0001 C CNN "Part#"
 	1    13500 14650
 	0    -1   -1   0
@@
 	16750 9025 16750 7775
 Connection ~ 16750 7775
+$Comp
+L Joker60-NoArrows-rescue:R_Small-Device-doddle60-rescue RL1
+U 1 1 5E5122FD
+P 11950 19925
+F 0 "RL1" V 11875 19925 31  0000 C CNN
+F 1 "620R" V 11950 19925 31  0000 C CNN
+F 2 "acheron_Components:R_SMD_1206" H 11950 19925 50  0001 C CNN
+F 3 "https://datasheet.lcsc.com/szlcsc/1810301439_UNI-ROYAL-Uniroyal-Elec-1206W4J0621T5E_C25391.pdf" H 11950 19925 50  0001 C CNN
+F 4 "C25391" H 11950 19925 50  0001 C CNN "LCSC Part#"
+F 5 "	UNI-ROYAL(Uniroyal Elec)" H 11950 19925 50  0001 C CNN "Mfr"
+F 6 "	1206W4J0621T5E" H 11950 19925 50  0001 C CNN "Part#"
+	1    11950 19925
+	1    0    0    -1
+$EndComp
 $EndSCHEMATC

Commit message: 8/29
Parts:
- removed CB1, CB4, CB6: 1µ, Capacitor_SMD:C_0402_1005Metric, symbol Joker60-NoArrows-rescue:C_Small-Device-doddle60-rescue
- removed CB10, CB9: 1µ, Capacitor_SMD:C_0805_2012Metric, symbol Joker60-NoArrows-rescue:C_Small-Device-doddle60-rescue
- removed CB2, CB3, CB5, CB8: 100n, Capacitor_SMD:C_0402_1005Metric, symbol Joker60-NoArrows-rescue:C_Small-Device-doddle60-rescue
- removed CB7: 100nF, Capacitor_SMD:C_0402_1005Metric, symbol Joker60-NoArrows-rescue:C_Small-Device-doddle60-rescue
- removed CRST1: 10u, Capacitor_SMD:C_0805_2012Metric_Pad1.15x1.40mm_HandSolder, symbol Joker60-NoArrows-rescue:C_Small-Device-doddle60-rescue
- removed CRST2: 4.7n, Capacitor_SMD:C_0805_2012Metric_Pad1.15x1.40mm_HandSolder, symbol Joker60-NoArrows-rescue:C_Small-Device-doddle60-rescue
- removed CSH1, CSH2: 4.7nF, Capacitor_SMD:C_0805_2012Metric, symbol Joker60-NoArrows-rescue:C_Small-Device-doddle60-rescue
- removed CSI1, CSO1: 1µ, Capacitor_SMD:C_0805_2012Metric_Pad1.15x1.40mm_HandSolder, symbol Joker60-NoArrows-rescue:C_Small-Device-doddle60-rescue
- removed CUSB1: 100n, Capacitor_SMD:C_0805_2012Metric_Pad1.15x1.40mm_HandSolder, symbol Joker60-NoArrows-rescue:C_Small-Device-doddle60-rescue
- removed DF1: SMF9.0CA, acheron_Components:D_SOD-123_Bidirectional, symbol Joker60-NoArrows-rescue:D_TVS-Device-doddle60-rescue
- removed DL1: 19-217/R6C-AL1M2VY/3T, LED_SMD:LED_0603_1608Metric, symbol Joker60-NoArrows-rescue:LED_Small-Device-doddle60-rescue
- removed DRST1: B0520LW, acheron_Components:D_SOD-123, symbol Joker60-NoArrows-rescue:D_Schottky-Device-doddle60-rescue
- removed DS1, DSH1: RB060M-60TR, acheron_Components:D_SOD-123, symbol Joker60-NoArrows-rescue:D_Schottky-Device-doddle60-rescue
- removed F1: 1A trip PTC, acheron_Components:Fuse_1812_4532, symbol Joker60-NoArrows-rescue:Polyfuse_Small-Device-doddle60-rescue
- removed G1: Doddle60Logo, doddle60Graphics:doddle60Logo, symbol Joker60-NoArrows-rescue:MountingHole-Mechanical-doddle60-rescue
- removed G2: OSHLogo, oshLogo:osh-logo, symbol Joker60-NoArrows-rescue:MountingHole-Mechanical-doddle60-rescue
- removed G3: Acheron Logo, acheron_Logos:acheronLong, symbol Joker60-NoArrows-rescue:MountingHole-Mechanical-doddle60-rescue
- removed G4: Doddle60Label, doddle60Graphics:doddle60Label, symbol Joker60-NoArrows-rescue:MountingHole-Mechanical-doddle60-rescue
- removed G5: LabelMask, doddle60Graphics:doddle60LabelMask, symbol Joker60-NoArrows-rescue:MountingHole-Mechanical-doddle60-rescue
- removed H1, H6: Half Side Hole, acheron_MountingHoles:halfSideHole, symbol Joker60-NoArrows-rescue:MountingHole-Mechanical-doddle60-rescue
- removed H10, H3, H4, H5, H7, H9: Oval Mounting Hole, acheron_MountingHoles:MoutingHole_Oval_7mm_5.0x2.5mm, symbol Joker60-NoArrows-rescue:MountingHole-Mechanical-doddle60-rescue
- removed H2: Mounting Hole, acheron_MountingHoles:MoutingHole_Oval_7mm_5.0x2.5mm, symbol Joker60-NoArrows-rescue:MountingHole-Mechanical-doddle60-rescue
- removed H8: Oval Mounting Hole, acheron_MountingHoles:MoutingHole_Oval_7mm_5.0x2.5mm, symbol Joker60-NoArrows-rescue:MountingHole_Pad-Mechanical-doddle60-rescue
- removed J1: TYPE-C-31-M12_13, acheron_Connectors:TYPE-C-31-M-12, symbol Joker60-NoArrows-rescue:TYPE-C-31-M12_13-acheronSymbols
- removed J2: Conn_01x14, acheron_Connectors:PinHeader_1x14_P2.54mm_Vertical, symbol Joker60-NoArrows-rescue:Conn_01x14-Connector_Generic-doddle60-rescue
- removed J3: Conn_ARM_JTAG_SWD_10, acheron_Connectors:Conn_ARM_JTAG_SWD_10, symbol Joker60-NoArrows-rescue:Conn_ARM_JTAG_SWD_10-Connector-doddle60-rescue
- removed L1: ACM2012-900-2P-T002, acheron_Components:ACM2012-2P, symbol Joker60-NoArrows-rescue:L_Core_Ferrite_Coupled_1423-acheronSymbols
- removed L2: MGFL1608F1R0MT-LF, Inductor_SMD:L_0603_1608Metric, symbol Joker60-NoArrows-rescue:L_Core_Ferrite-Device-doddle60-rescue
- removed L3: CMI322513U1R0KT, Inductor_SMD:L_1210_3225Metric, symbol Joker60-NoArrows-rescue:L_Core_Ferrite-Device-doddle60-rescue
- removed QRST1: DTC123J, Package_TO_SOT_SMD:SOT-23, symbol Joker60-NoArrows-rescue:DTC123J-Transistor_BJT-doddle60-rescue
- removed RL1: 620R, acheron_Components:R_SMD_1206, symbol Joker60-NoArrows-rescue:R_Small-Device-doddle60-rescue
- removed RPU1: 1.5k, acheron_Components:R_SMD_1206, symbol Joker60-NoArrows-rescue:R_Small-Device-doddle60-rescue
- removed RRST1, RSI1, RSO1: 100k, acheron_Components:R_SMD_1206, symbol Joker60-NoArrows-rescue:R_Small-Device-doddle60-rescue
- removed RSH1, RSH2: 1M, acheron_Components:R_SMD_1206, symbol Joker60-NoArrows-rescue:R_Small-Device-doddle60-rescue
- removed RVDD1: R010 1%, acheron_Components:R_SMD_1206, symbol Joker60-NoArrows-rescue:R_Small-Device-doddle60-rescue
- removed SWRST1: SW_Push, acheron_Hardware:smdPushBtn, symbol Joker60-NoArrows-rescue:SW_Push-Switch-doddle60-rescue
- removed U1: STM32F072-LQFP48, acheron_Components:LQFP-48_7x7mm_P0.5mm, symbol Joker60-NoArrows-rescue:STM32F072-LQFP48-acheronSymbols
- removed U2: USBLC6-2SC6, acheron_Components:SOT-23-6, symbol Joker60-NoArrows-rescue:USBLC6-2SC6-Power_Protection-doddle60-rescue
- removed U3: MCP1700-3302E_SOT23, Package_TO_SOT_SMD:SOT-23, symbol Joker60-NoArrows-rescue:MCP1700-3302E_SOT23-Regulator_Linear-doddle60-rescue
- added C1: 1uF, Capacitor_SMD:C_0603_1608Metric, symbol Device:C_Small
- added C2, C3, C4: 0.1uF, Capacitor_SMD:C_0603_1608Metric, symbol Device:C_Small
- added C5: 10uF, Capacitor_SMD:C_0603_1608Metric, symbol Device:C_Small
- added F1: Polyfuse_Small, Fuse:Fuse_0805_2012Metric, symbol Device:Polyfuse_Small
- added J2: Conn_02x03_Odd_Even, Connector_PinHeader_2.54mm:PinHeader_2x03_P2.54mm_Vertical, symbol Connector_Generic:Conn_02x03_Odd_Even
- added R1, R2: 22Ω, Resistor_SMD:R_0603_1608Metric, symbol Device:R_Small
- added R3, R4: 10kΩ, Resistor_SMD:R_0603_1608Metric, symbol Device:R_Small
- added SW118: SW_PUSH, random-keyboard-parts:SKQG-1155865, symbol kbd:SW_PUSH
- added U1: SRV05-4, Package_TO_SOT_SMD:SOT-23-6, symbol Power_Protection:SRV05-4
- added U2: ATmega32U4-MU, Package_DFN_QFN:QFN-44-1EP_7x7mm_P0.5mm_EP5.2x5.2mm, symbol MCU_Microchip_ATmega:ATmega32U4-MU
- added USB1: HRO-TYPE-C-31-M-12, Keebio-Parts:HRO-TYPE-C-31-M-12-Assembly, symbol keebio:HRO-TYPE-C-31-M-12
- added Y1: Resonator_Small, proj_local:Resonator_SMD_muRata_CSTxExxV-3Pin_3.0x1.1mm_HandSoldering_Compact, symbol Device:Resonator_Small
- RCC1, RCC2: footprint acheron_Components:R_SMD_1206 -> Resistor_SMD:R_0805_2012Metric
- SW96: footprint acheron_MX_SolderMask:MX200R -> acheron_MX_SolderMask:MX200
Connections:
- net Col1: now also U2.31 (PC6)
- net Col10: now also U2.19 (PD1)
- net Col11: now also U2.18 (PD0)
- net Col12: now also U2.12 (PB7)
- net Col13: now also J2.1 (Pin_1), U2.11 (PB3)
- net Col14: now also J2.4 (Pin_4), U2.10 (PB2)
- net Col15: now also U2.8 (PB0)
- net Col2: now also U2.39 (PF4)
- net Col3: now also U2.28 (PB4)
- net Col4: now also U2.27 (PD7)
- net Col5: now also U2.26 (PD6)
- net Col6: now also U2.25 (PD4)
- net Col7: now also U2.22 (PD5)
- net Col8: now also U2.21 (PD3)
- net Col9: now also U2.20 (PD2)
- net D+: now also R2.2, U1.6 (IO4), USB1.6 (DP1), USB1.8 (DP2)
- net D-: now also R1.2, U1.1 (IO1), USB1.5 (DN2), USB1.7 (DN1)
- net GND: now also C1.2, C2.2, C3.2, C4.2, C5.2, J2.6 (Pin_6), R4.1, SW118.1, U1.2 (VN), U2.15 (GND), U2.23 (GND), U2.35 (GND), U2.43 (GND), U2.45 (GND), U2.5 (UGND), USB1.1 (GND), USB1.12 (GND), USB1.13 (SHIELD), Y1.2
- net Row1: now also J2.3 (Pin_3), U2.9 (PB1)
- net Row2: now also U2.41 (PF0)
- net Row3: now also U2.29 (PB5)
- net Row4: now also U2.30 (PB6)
- net Row5: now also U2.32 (PC7)
- net at RCC2.2: now also USB1.4 (CC1)
- net at RCC1.2: now also USB1.10 (CC2)
- new net: J2.5 (Pin_5), R3.2, SW118.2, U2.13 (~RESET)
- new net: U2.16 (XTAL2), Y1.3
- new net: U2.17 (XTAL1), Y1.1
- new net: R1.1, U2.3 (D-)
- new net: R4.2, U2.33 (~HWB~/PE2)
- new net: R2.1, U2.4 (D+)
- new net: C1.1, U2.6 (UCAP)
- new net +5V: C2.1, C3.1, C4.1, C5.1, F1.1, J2.2 (Pin_2), R3.1, U2.14 (VCC), U2.2 (UVCC), U2.24 (AVCC), U2.34 (VCC), U2.44 (AVCC), U2.7 (VBUS)
- new net VCC: F1.2, U1.5 (VP), USB1.11 (VBUS), USB1.2 (VBUS)
- no-connect marks 4 -> 3
Other:
- note removed: "CBx are the bypass capacitors. Their value is specified in reference [2]."
- note removed: "Case ESD"
- note removed: "Extra pins"
- note removed: "Hard reset circuit"
- note removed: "Logos and flags"
- note removed: "MCU"
- note removed: "Mounting holes"
- note removed: "Power supply and protection circuit"
- note removed: "REFERENCES"
- note removed: "Serial programming"
- note removed: "Shield"
- note removed: "Switch matrix"
- note removed: "USB Connector"
- note removed: "USD ESD"
- note removed: "[1] STM32F072x8 / STM32F072xB datasheet"
- note removed: "[2] AN4080 Application note"
- note removed: "https://www.st.com/content/ccc/resource/technical/document/application_note/c9/19/d7/b8/6b/0e/4c/d3/DM00051986.pdf/files/DM00051986.pdf/jcr:content/translations/en.DM00051986.pdf"
- note removed: "https://www.st.com/resource/en/datasheet/stm32f072rb.pdf"
- moved on the sheet: RCC1, RCC2
