File: PCB/Joker60-NoArrows.sch (KiCad schematic (older format))
At the start: 205 parts, among them J2 Conn_02x03_Odd_Even, SW1 ESC, SW10 9, SW100 SPACE_625, SW101 HENKAN_100, SW102 RALT_100, SW103 RALT_100, SW104 RGUI_100, SW105 RCTRL_100, SW106 LGUI_100, SW107 LALT_125, SW108 MUHENKAN_100, SW109 SPACE_450, SW11 0, SW110 HENKAN_125, SW111 HENKAN_125, SW112 HENKAN_125, SW113 RALT_100, SW114 RALT_125, SW115 RCTRL_100, SW116 RCTRL_100, SW117 RCTRL_100, SW118 SW_PUSH, SW12 -_, SW13 +=, SW14 2U BKSP, SW15 TAB_150, SW16 Q, SW17 W, SW18 E, SW19 R, SW2 1, SW20 T, SW21 Y, SW22 U, SW23 I, SW24 O, SW25 P, SW26 [{, SW27 ]}, SW28 1U_RBKSP, SW29 CAPS_175, SW3 2, SW30 A, SW31 S, SW32 D, SW33 F, SW34 G, SW35 H, SW36 J, SW37 K, SW38 L, SW39 :;, SW4 3, SW40 @', SW41 ~~#, SW42 LSHIFT_125, SW43 |\\, SW44 Z, SW45 X, SW46 C, SW47 V, SW48 B, SW49 N, SW5 4, SW50 M, SW51 <,, SW52 >., SW53 ?/, SW54 LCTRL_100, SW55 LGUI_125, SW56 LALT_100, SW57 SPACE_275, SW58 RALT_125, SW59 RGUI_125, SW6 5, SW60 RCTRL_125, SW61 LGUI_125, SW62 LALT_125, SW63 STEPPED_CAPS_125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

Commit message: 10/7
Connections:
- net Col15 is gone; now on net Col14: SW76.1 (Col), U2.8 (PB0)
- net Row5 is gone; now on net Row4: D54.1 (K), D55.1 (K), D56.1 (K), D57.1 (K), D58.1 (K), D59.1 (K), D60.1 (K), D61.1 (K), D64.1 (K), D66.1 (K), D67.1 (K), D69.1 (K), D70.1 (K), U2.32 (PC7)
- net Col1: now also SW106.1 (Col), SW16.1 (Col), SW2.1 (Col), SW30.1 (Col), SW43.1 (Col), SW54.1 (Col), SW55.1 (Col), SW69.1 (Col), U2.39 (PF4); no longer SW1.1 (Col), SW15.1 (Col), SW29.1 (Col), SW42.1 (Col), SW61.1 (Col), SW63.1 (Col), SW66.1 (Col), SW73.1 (Col), SW98.1 (Col), U2.31 (PC6)
- net Col10: now also SW102.1 (Col), SW11.1 (Col), SW112.1 (Col), SW25.1 (Col), SW39.1 (Col), SW52.1 (Col), SW58.1 (Col), SW84.1 (Col), SW94.1 (Col), U2.18 (PD0); no longer SW10.1 (Col), SW101.1 (Col), SW111.1 (Col), SW24.1 (Col), SW38.1 (Col), SW51.1 (Col), SW68.1 (Col), SW83.1 (Col), SW93.1 (Col), U2.19 (PD1)
- net Col11: now also SW103.1 (Col), SW113.1 (Col), SW115.1 (Col), SW12.1 (Col), SW26.1 (Col), SW40.1 (Col), SW53.1 (Col), SW59.1 (Col), SW95.1 (Col), U2.12 (PB7); no longer SW102.1 (Col), SW11.1 (Col), SW112.1 (Col), SW25.1 (Col), SW39.1 (Col), SW52.1 (Col), SW58.1 (Col), SW84.1 (Col), SW94.1 (Col), U2.18 (PD0)
- net Col12: now also J2.1 (Pin_1), SW104.1 (Col), SW116.1 (Col), SW13.1 (Col), SW27.1 (Col), SW41.1 (Col), SW74.1 (Col), SW78.1 (Col), SW96.1 (Col), SW99.1 (Col), U2.11 (PB3); no longer SW103.1 (Col), SW113.1 (Col), SW115.1 (Col), SW12.1 (Col), SW26.1 (Col), SW40.1 (Col), SW53.1 (Col), SW59.1 (Col), SW95.1 (Col), U2.12 (PB7)
- net Col13: now also J2.4 (Pin_4), SW105.1 (Col), SW114.1 (Col), SW117.1 (Col), SW14.1 (Col), SW28.1 (Col), SW60.1 (Col), SW64.1 (Col), SW65.1 (Col), SW72.1 (Col), SW75.1 (Col), SW77.1 (Col), SW79.1 (Col), SW97.1 (Col), U2.10 (PB2); no longer J2.1 (Pin_1), SW104.1 (Col), SW116.1 (Col), SW13.1 (Col), SW27.1 (Col), SW41.1 (Col), SW74.1 (Col), SW78.1 (Col), SW96.1 (Col), SW99.1 (Col), U2.11 (PB3)
- net Col14: no longer J2.4 (Pin_4), SW105.1 (Col), SW114.1 (Col), SW117.1 (Col), SW14.1 (Col), SW28.1 (Col), SW60.1 (Col), SW64.1 (Col), SW65.1 (Col), SW72.1 (Col), SW75.1 (Col), SW77.1 (Col), SW79.1 (Col), SW97.1 (Col), U2.10 (PB2)
- net Col2: now also SW107.1 (Col), SW17.1 (Col), SW3.1 (Col), SW31.1 (Col), SW44.1 (Col), SW56.1 (Col), SW62.1 (Col), SW71.1 (Col), U2.28 (PB4); no longer SW106.1 (Col), SW16.1 (Col), SW2.1 (Col), SW30.1 (Col), SW43.1 (Col), SW54.1 (Col), SW55.1 (Col), SW69.1 (Col), U2.39 (PF4)
- net Col3: now also SW108.1 (Col), SW18.1 (Col), SW32.1 (Col), SW4.1 (Col), SW45.1 (Col), SW67.1 (Col), SW81.1 (Col), SW85.1 (Col), U2.27 (PD7); no longer SW107.1 (Col), SW17.1 (Col), SW3.1 (Col), SW31.1 (Col), SW44.1 (Col), SW56.1 (Col), SW62.1 (Col), SW71.1 (Col), U2.28 (PB4)
- net Col4: now also SW19.1 (Col), SW33.1 (Col), SW46.1 (Col), SW5.1 (Col), SW87.1 (Col), U2.26 (PD6); no longer SW108.1 (Col), SW18.1 (Col), SW32.1 (Col), SW4.1 (Col), SW45.1 (Col), SW67.1 (Col), SW81.1 (Col), SW85.1 (Col), U2.27 (PD7)
- net Col5: now also SW20.1 (Col), SW34.1 (Col), SW47.1 (Col), SW6.1 (Col), SW70.1 (Col), SW88.1 (Col), U2.25 (PD4); no longer SW19.1 (Col), SW33.1 (Col), SW46.1 (Col), SW5.1 (Col), SW87.1 (Col), U2.26 (PD6)
- net Col6: now also SW100.1 (Col), SW109.1 (Col), SW21.1 (Col), SW35.1 (Col), SW48.1 (Col), SW57.1 (Col), SW7.1 (Col), SW86.1 (Col), SW90.1 (Col), U2.22 (PD5); no longer SW20.1 (Col), SW34.1 (Col), SW47.1 (Col), SW6.1 (Col), SW70.1 (Col), SW88.1 (Col), U2.25 (PD4)
- net Col7: now also SW22.1 (Col), SW36.1 (Col), SW49.1 (Col), SW8.1 (Col), SW89.1 (Col), SW91.1 (Col), U2.21 (PD3); no longer SW100.1 (Col), SW109.1 (Col), SW21.1 (Col), SW35.1 (Col), SW48.1 (Col), SW57.1 (Col), SW7.1 (Col), SW86.1 (Col), SW90.1 (Col), U2.22 (PD5)
- net Col8: now also SW110.1 (Col), SW23.1 (Col), SW37.1 (Col), SW50.1 (Col), SW80.1 (Col), SW82.1 (Col), SW9.1 (Col), SW92.1 (Col), U2.20 (PD2); no longer SW22.1 (Col), SW36.1 (Col), SW49.1 (Col), SW8.1 (Col), SW89.1 (Col), SW91.1 (Col), U2.21 (PD3)
- net Col9: now also SW10.1 (Col), SW101.1 (Col), SW111.1 (Col), SW24.1 (Col), SW38.1 (Col), SW51.1 (Col), SW68.1 (Col), SW83.1 (Col), SW93.1 (Col), U2.19 (PD1); no longer SW110.1 (Col), SW23.1 (Col), SW37.1 (Col), SW50.1 (Col), SW80.1 (Col), SW82.1 (Col), SW9.1 (Col), SW92.1 (Col), U2.20 (PD2)
- net Row1: now also D15.1 (K), D16.1 (K), D17.1 (K), D18.1 (K), D19.1 (K), D20.1 (K), D21.1 (K), D22.1 (K), D23.1 (K), D24.1 (K), D25.1 (K), D26.1 (K), D27.1 (K), D28.1 (K), D68.1 (K), U2.41 (PF0); no longer D1.1 (K), D10.1 (K), D11.1 (K), D12.1 (K), D13.1 (K), D14.1 (K), D2.1 (K), D3.1 (K), D4.1 (K), D5.1 (K), D6.1 (K), D7.1 (K), D8.1 (K), D9.1 (K), J2.3 (Pin_3), U2.9 (PB1)
- net Row2: now also D29.1 (K), D30.1 (K), D31.1 (K), D32.1 (K), D33.1 (K), D34.1 (K), D35.1 (K), D36.1 (K), D37.1 (K), D38.1 (K), D39.1 (K), D40.1 (K), D41.1 (K), D65.1 (K), U2.29 (PB5); no longer D15.1 (K), D16.1 (K), D17.1 (K), D18.1 (K), D19.1 (K), D20.1 (K), D21.1 (K), D22.1 (K), D23.1 (K), D24.1 (K), D25.1 (K), D26.1 (K), D27.1 (K), D28.1 (K), D68.1 (K), U2.41 (PF0)
- net Row3: now also D42.1 (K), D43.1 (K), D44.1 (K), D45.1 (K), D46.1 (K), D47.1 (K), D48.1 (K), D49.1 (K), D50.1 (K), D51.1 (K), D52.1 (K), D53.1 (K), D62.1 (K), D63.1 (K), U2.30 (PB6); no longer D29.1 (K), D30.1 (K), D31.1 (K), D32.1 (K), D33.1 (K), D34.1 (K), D35.1 (K), D36.1 (K), D37.1 (K), D38.1 (K), D39.1 (K), D40.1 (K), D41.1 (K), D65.1 (K), U2.29 (PB5)
- net Row4: no longer D42.1 (K), D43.1 (K), D44.1 (K), D45.1 (K), D46.1 (K), D47.1 (K), D48.1 (K), D49.1 (K), D50.1 (K), D51.1 (K), D52.1 (K), D53.1 (K), D62.1 (K), D63.1 (K), U2.30 (PB6)
- new net Col0: SW1.1 (Col), SW15.1 (Col), SW29.1 (Col), SW42.1 (Col), SW61.1 (Col), SW63.1 (Col), SW66.1 (Col), SW73.1 (Col), SW98.1 (Col), U2.31 (PC6)
- new net Row0: D1.1 (K), D10.1 (K), D11.1 (K), D12.1 (K), D13.1 (K), D14.1 (K), D2.1 (K), D3.1 (K), D4.1 (K), D5.1 (K), D6.1 (K), D7.1 (K), D8.1 (K), D9.1 (K), J2.3 (Pin_3), U2.9 (PB1)
Changed lines of the file:
@@
 $EndDescr
 Text GLabel 2500 3025 0    50   Input ~ 0
-Row2
-Text GLabel 2500 2050 0    50   Input ~ 0
 Row1
+Text GLabel 2500 2050 0    50   Input ~ 0
+Row0
 $Comp
 L Joker60-NoArrows-rescue:D-Device-doddle60-rescue D13
@@
 $EndComp
 Text GLabel 13850 1700 1    50   Input ~ 0
-Col12
-Text GLabel 12850 1700 1    50   Input ~ 0
 Col11
-Text GLabel 11850 1700 1    50   Input ~ 0
+Text GLabel 12850 1700 1    50   Input ~ 0
 Col10
-Text GLabel 10850 1700 1    50   Input ~ 0
+Text GLabel 11850 1700 1    50   Input ~ 0
 Col9
-Text GLabel 9850 1700 1    50   Input ~ 0
+Text GLabel 10850 1700 1    50   Input ~ 0
 Col8
-Text GLabel 8850 1700 1    50   Input ~ 0
+Text GLabel 9850 1700 1    50   Input ~ 0
 Col7
-Text GLabel 7850 1700 1    50   Input ~ 0
+Text GLabel 8850 1700 1    50   Input ~ 0
 Col6
-Text GLabel 6850 1700 1    50   Input ~ 0
+Text GLabel 7850 1700 1    50   Input ~ 0
 Col5
-Text GLabel 5850 1700 1    50   Input ~ 0
+Text GLabel 6850 1700 1    50   Input ~ 0
 Col4
-Text GLabel 4850 1700 1    50   Input ~ 0
+Text GLabel 5850 1700 1    50   Input ~ 0
 Col3
-Text GLabel 3850 1700 1    50   Input ~ 0
+Text GLabel 4850 1700 1    50   Input ~ 0
 Col2
-Text GLabel 2850 1700 1    50   Input ~ 0
+Text GLabel 3850 1700 1    50   Input ~ 0
 Col1
+Text GLabel 2850 1700 1    50   Input ~ 0
+Col0
 Wire Wire Line
 	3000 2700 2850 2700
 Text GLabel 14850 1700 1    50   Input ~ 0
-Col13
+Col12
 $Comp
 L Joker60-NoArrows-rescue:D-Device-doddle60-rescue D7
@@
 $EndComp
 Text GLabel 15850 1700 1    50   Input ~ 0
-Col14
+Col13
 Wire Wire Line
 	15350 2050 16350 2050
@@
 	4850 2700 4850 3675
 Text GLabel 2500 4000 0    50   Input ~ 0
-Row3
+Row2
 Wire Wire Line
 	3000 4650 2850 4650
@@
 	4850 3675 4850 4650
 Text GLabel 2500 4975 0    50   Input ~ 0
-Row4
+Row3
 Wire Wire Line
 	3000 5625 2850 5625
@@
 	3350 4000 4350 4000
 Text GLabel 2500 5950 0    50   Input ~ 0
-Row5
+Row4
 Wire Wire Line
 	3000 6600 2850 6600
@@
 Connection ~ 16350 3025
 Text GLabel 16800 1700 1    50   Input ~ 0
-Col15
+Col14
 Wire Wire Line
 	16800 3675 16800 1700
@@
 	14025 11225 13850 11225
 Text GLabel 16750 11325 2    50   Input ~ 0
-Row1
+Row0
 Text GLabel 15675 13625 2    50   Input ~ 0
-Row2
+Row1
 Text GLabel 15675 11725 2    50   Input ~ 0
-Row3
+Row2
 Text GLabel 15675 11825 2    50   Input ~ 0
-Row4
+Row3
 Text GLabel 15675 12225 2    50   Input ~ 0
-Row5
+Row4
 Text GLabel 15675 12125 2    50   Input ~ 0
-Col1
+Col0
 Text GLabel 15675 13825 2    50   Input ~ 0
-Col2
+Col1
 Text GLabel 15675 11625 2    50   Input ~ 0
-Col3
+Col2
 Text GLabel 15675 13125 2    50   Input ~ 0
-Col4
+Col3
 Text GLabel 15675 13025 2    50   Input ~ 0
-Col5
+Col4
 Text GLabel 15675 12825 2    50   Input ~ 0
-Col6
+Col5
 Text GLabel 15675 12925 2    50   Input ~ 0
-Col7
+Col6
 Text GLabel 15675 12725 2    50   Input ~ 0
-Col8
+Col7
 Text GLabel 15675 12625 2    50   Input ~ 0
-Col9
+Col8
 Text GLabel 15675 12525 2    50   Input ~ 0
-Col10
+Col9
 Text GLabel 15675 12425 2    50   Input ~ 0
-Col11
+Col10
 Wire Wire Line
 	15675 13325 16000 13325
@@
 $EndComp
 Text GLabel 15675 11925 2    50   Input ~ 0
-Col12
+Col11
 Text GLabel 16750 11525 2    50   Input ~ 0
-Col13
+Col12
 Text GLabel 16750 11425 2    50   Input ~ 0
-Col14
+Col13
 Text GLabel 15675 11225 2    50   Input ~ 0
-Col15
+Col14
 $Comp
 L Power_Protection:SRV05-4 U1
